File: pcb/trackpad.kicad_pcb (KiCad board)
At the start: 4 copper layers, 79 x 49 mm, 31 parts, among them J1 Conn_01x06, U1 IQS550

Commit message: Fix silkscreen
Other:
- board text added: "GR-Trackpad65"
- board text removed: "TPS65 Clone"
